File: Nucleo-F767-Base-Board.kicad_pcb (KiCad board)
At the start: 2 copper layers, 120 x 130 mm, 81 parts, among them IC1 TLP152, IC2 TLP152, IC3 TLP152, IC4 TLP152, J1 Conn_01x02_Pin, J14 Conn_01x02_Pin, J15 Conn_01x02_Pin, J16 Conn_01x02_Pin, J17 Conn_01x02_Pin, J2 Conn_01x02_Pin, J20 Conn_01x03_Pin, J21 Conn_01x03_Pin, J24 Conn_01x03_Pin, J25 Conn_01x03_Pin, J3 Conn_01x02_Pin, J4 Conn_01x02_Pin, J5 Conn_01x02_Pin, J6 Conn_01x02_Pin, J7 Conn_01x02_Pin, J8 Conn_01x02_Pin, J9 Conn_01x02_Pin, Q1 RS6G120BGTB1, Q2 RS6G120BGTB1, Q3 RS6G120BGTB1, Q4 RS6G120BGTB1, SW1 SW_Push, SW2 SW_Push, U1 MC78M09CDTRKG, U4 TBD62783A, U5 TPS5450, U6 MCP2551-I-P

Commit message: Update.
Parts:
- moved J1 0.50 mm to (72.2, 143.0)
Connections:
- A1 pad CN10_28: SW1 -> PWM1
- A1 pad CN10_6: unconnected-(A1D-D5/TIMER_A_PWM2-PadCN10_6) -> SW1
- A1 pad CN8_2: PWM2 -> unconnected-(A1B-D43/SDMMC_D0-PadCN8_2)
- A1 pad CN8_4: PWM1 -> unconnected-(A1B-D44/SDMMC_D1/I2S_A_CKIN-PadCN8_4)
- A1 pad CN9_28: unconnected-(A1C-D63/SAI_B_FS-PadCN9_28) -> PWM2
Routing:
- net PWM1: track 83.3 -> 165.5 mm
- net PWM2: track 89.5 -> 158.5 mm
- net SW1: track 130.2 -> 158.2 mm
- net +9V: track 140.9 -> 145.4 mm

Commit message: Fixed
Parts:
- removed R11, R13: 1k, Resistor_SMD:R_0603_1608Metric
- removed R12, R14: 1.5k, Resistor_SMD:R_0603_1608Metric
- moved J20 13.0 mm to (49.2, 64.7)
- moved J21 13.0 mm to (49.2, 51.6)
- moved R1 11.2 mm to (59.1, 131.8)
- moved R3 11.2 mm to (59.1, 116.8)
- moved R5 11.2 mm to (59.1, 101.8)
- moved R7 11.1 mm to (58.9, 86.9)
- moved R2 10.4 mm to (57.1, 131.8), turned to -90 degrees
- moved R4 10.4 mm to (57.1, 116.8), turned to -90 degrees
- moved R6 10.3 mm to (57.1, 101.8), turned to -90 degrees
- moved R8 10.3 mm to (56.9, 86.9), turned to -90 degrees
- moved R25 3.90 mm to (62.4, 46.6), turned to -90 degrees
- moved R24 3.79 mm to (66.0, 46.6), turned to -90 degrees
- moved R23 3.71 mm to (69.6, 46.6), turned to -90 degrees
- moved R20 3.69 mm to (73.2, 46.6), turned to -90 degrees
- moved D12 3.36 mm to (62.4, 50.0), turned to 90 degrees
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Connections:
- A1 pad CN8_2: unconnected-(A1B-D43/SDMMC_D0-PadCN8_2) -> PWM3
- A1 pad CN8_4: unconnected-(A1B-D44/SDMMC_D1/I2S_A_CKIN-PadCN8_4) -> PWM4
- A1 pad CN9_1: ADC2 -> unconnected-(A1C-A0/ADC123_IN3-PadCN9_1)
- A1 pad CN9_3: ADC1 -> unconnected-(A1C-A1/ADC123_IN10-PadCN9_3)
- D10 pad 1: AIRIN2 -> GND
- D11 pad 1: AIRIN3 -> GND
- D12 pad 1: AIRIN4 -> GND
- D13 pad 1: MOS_IN1 -> GND
- D14 pad 1: MOS_IN2 -> GND
- D15 pad 1: MOS_IN3 -> GND
- D16 pad 1: MOS_IN4 -> GND
- D9 pad 1: AIRIN1 -> GND
- J1 pad 1: VDD -> GND
- J1 pad 2: GND -> VDD
- J14 pad 1: AIROUT1 -> GND
- J14 pad 2: GND -> AIROUT1
- J15 pad 1: AIROUT2 -> GND
- J15 pad 2: GND -> AIROUT2
- J16 pad 1: AIROUT3 -> GND
- J16 pad 2: GND -> AIROUT3
- J17 pad 1: AIROUT4 -> GND
- J17 pad 2: GND -> AIROUT4
- J20 pad 2: Net-(J20-Pin_2) -> PWM3
- J21 pad 2: Net-(J21-Pin_2) -> PWM4
- J4 pad 1: VDD -> Net-(D1-A)
- J4 pad 2: Net-(D1-A) -> VDD
- J5 pad 1: VDD -> Net-(D2-A)
- J5 pad 2: Net-(D2-A) -> VDD
- J6 pad 1: VDD -> Net-(D3-A)
- J6 pad 2: Net-(D3-A) -> VDD
- J7 pad 1: VDD -> Net-(D4-A)
- J7 pad 2: Net-(D4-A) -> VDD
- R15 pad 1: +3.3V -> MOS_IN1
- R16 pad 1: +3.3V -> MOS_IN2
- R17 pad 1: +3.3V -> MOS_IN3
- R18 pad 1: +3.3V -> MOS_IN4
- R20 pad 1: +3.3V -> AIRIN1
- R23 pad 1: +3.3V -> AIRIN2
- R24 pad 1: +3.3V -> AIRIN3
- R25 pad 1: +3.3V -> AIRIN4
Routing:
- net ADC1: track 86.4 -> 0.00 mm
- net +3.3V: track 116.1 -> 44.5 mm, vias 6 -> 3
- net PWM4: track 0.00 -> 63.6 mm
- net ADC2: track 56.7 -> 0.00 mm
- net PWM3: track 0.00 -> 46.3 mm
- net Net-(IC4-Vo): track 20.9 -> 32.9 mm
- net Net-(IC3-Vo): track 11.0 -> 22.0 mm
- net MOS_IN4: track 43.8 -> 33.0 mm
- net Net-(IC1-Vo): track 16.0 -> 5.54 mm
- net VDD: track 127.1 -> 117.9 mm
- net GND: track 54.5 -> 63.3 mm, vias 54 -> 58
- net Net-(J20-Pin_2): track 7.45 -> 0.00 mm
- net Net-(J21-Pin_2): track 7.30 -> 0.00 mm
- net Net-(IC2-Vo): track 6.01 -> 12.6 mm
- net MOS_IN3: track 40.5 -> 35.4 mm
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Other:
- board text added: "CatchRobo2024 Board 1.1 Designer: Xinjia Li (FF21)"
- board text removed: "CatchRobo2024 Board Designer: Xinjia Li (FF21)"
