File: Nucleo-F767-Base-Board.kicad_sch (KiCad schematic)
At the start: 79 parts, among them IC1 TLP152, IC2 TLP152, IC3 TLP152, IC4 TLP152, J1 Conn_01x02_Pin, J14 Conn_01x02_Pin, J15 Conn_01x02_Pin, J16 Conn_01x02_Pin, J17 Conn_01x02_Pin, J2 Conn_01x02_Pin, J20 Conn_01x03_Pin, J21 Conn_01x03_Pin, J24 Conn_01x03_Pin, J25 Conn_01x03_Pin, J3 Conn_01x02_Pin, J4 Conn_01x02_Pin, J5 Conn_01x02_Pin, J6 Conn_01x02_Pin, J7 Conn_01x02_Pin, J8 Conn_01x02_Pin, J9 Conn_01x02_Pin, Q1 RS6G120BGTB1, Q2 RS6G120BGTB1, Q3 RS6G120BGTB1, Q4 RS6G120BGTB1, SW1 SW_Push, SW2 SW_Push, U1 MC78M09CDTRKG, U4 TBD62783A, U5 TPS5450, U6 MCP2551-I-P

Commit message: Fixed
Parts:
- removed R11, R13: 1k, Resistor_SMD:R_0603_1608Metric, symbol Device:R
- removed R12, R14: 1.5k, Resistor_SMD:R_0603_1608Metric, symbol Device:R
Connections:
- net +3.3V: no longer R15.1, R16.1, R17.1, R18.1, R20.1, R23.1, R24.1, R25.1
- net AIRIN1: now also R20.1; no longer D9.1 (K)
- net AIRIN2: now also R23.1; no longer D10.1 (K)
- net AIRIN3: now also R24.1; no longer D11.1 (K)
- net AIRIN4: now also R25.1; no longer D12.1 (K)
- net AIROUT1: now also J14.2 (Pin_2); no longer J14.1 (Pin_1)
- net AIROUT2: now also J15.2 (Pin_2); no longer J15.1 (Pin_1)
- net AIROUT3: now also J16.2 (Pin_2); no longer J16.1 (Pin_1)
- net AIROUT4: now also J17.2 (Pin_2); no longer J17.1 (Pin_1)
- net GND: now also D10.1 (K), D11.1 (K), D12.1 (K), D13.1 (K), D14.1 (K), D15.1 (K), D16.1 (K), D9.1 (K), J1.1 (Pin_1), J14.1 (Pin_1), J15.1 (Pin_1), J16.1 (Pin_1), J17.1 (Pin_1); no longer J1.2 (Pin_2), J14.2 (Pin_2), J15.2 (Pin_2), J16.2 (Pin_2), J17.2 (Pin_2)
- net MOS_IN1: now also R15.1; no longer D13.1 (K)
- net MOS_IN2: now also R16.1; no longer D14.1 (K)
- net MOS_IN3: now also R17.1; no longer D15.1 (K)
- net MOS_IN4: now also R18.1; no longer D16.1 (K)
- net VDD: now also J1.2 (Pin_2), J4.2 (Pin_2), J5.2 (Pin_2), J6.2 (Pin_2), J7.2 (Pin_2); no longer J1.1 (Pin_1), J4.1 (Pin_1), J5.1 (Pin_1), J6.1 (Pin_1), J7.1 (Pin_1)
- net at D1.2 (A), Q1.1 (D): now also J4.1 (Pin_1); no longer J4.2 (Pin_2)
- net at D2.2 (A), Q2.1 (D): now also J5.1 (Pin_1); no longer J5.2 (Pin_2)
- net at D3.2 (A), Q3.1 (D): now also J6.1 (Pin_1); no longer J6.2 (Pin_2)
- net at D4.2 (A), Q4.1 (D): now also J7.1 (Pin_1); no longer J7.2 (Pin_2)
- net PWM4: now reaches J21.2 (Pin_2)
- net PWM3: now reaches J20.2 (Pin_2)
Other:
- moved on the sheet: D13, D14, D15, D16, J1, J20, J21, J4, J5, J6, J7, R15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
