File: nucleo.kicad_sch (KiCad schematic)
At the start: 1 part

Commit message: Update.
Connections:
- net PWM1: now also A1.CN10_28 (D38/IO); no longer A1.CN8_4 (D44/SDMMC_D1/I2S_A_CKIN)
- net PWM2: now also A1.CN9_28 (D63/SAI_B_FS); no longer A1.CN8_2 (D43/SDMMC_D0)
- net SW1: now also A1.CN10_6 (D5/TIMER_A_PWM2); no longer A1.CN10_28 (D38/IO)

Commit message: Fixed
Connections:
- net PWM3: now reaches A1.CN8_2 (D43/SDMMC_D0)
- net PWM4: now reaches A1.CN8_4 (D44/SDMMC_D1/I2S_A_CKIN)
- net ADC1: no longer names the net of A1.CN9_3 (A1/ADC123_IN10)
- net ADC2: no longer names the net of A1.CN9_1 (A0/ADC123_IN3)
Changed lines of the file:
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@@
-	(wire
-		(pts
-			(xy 55.88 102.87) (xy 58.42 102.87)
-		)
-		(stroke
-			(width 0)
-			(type default)
-		)
-	)
 	(wire
 		(pts
@@
 	(wire
 		(pts
+			(xy 166.37 55.88) (xy 168.91 55.88)
+		)
+		(stroke
+			(width 0)
+			(type default)
+		)
+	)
+	(wire
+		(pts
 			(xy 234.95 128.27) (xy 232.41 128.27)
 		)
@@
 	(wire
 		(pts
+			(xy 166.37 58.42) (xy 168.91 58.42)
+		)
+		(stroke
+			(width 0)
+			(type default)
+		)
+	)
+	(wire
+		(pts
 			(xy 234.95 153.67) (xy 234.95 151.13)
 		)
@@
 	(wire
 		(pts
-			(xy 55.88 105.41) (xy 58.42 105.41)
-		)
-		(stroke
-			(width 0)
-			(type default)
-		)
-	)
-	(wire
-		(pts
 			(xy 121.92 148.59) (xy 121.92 153.67)
 		)
@@
 		)
 	)
-	(global_label "ADC2"
-		(shape input)
-		(at 55.88 102.87 180)
-		(fields_autoplaced yes)
-		(effects
-			(font
-				(size 0.762 0.762)
-			)
-			(justify right)
-		)
-		(property "Intersheetrefs" "${INTERSHEET_REFS}"
-			(at 51.1858 102.87 0)
-			(effects
-				(font
-					(size 1.27 1.27)
-				)
-				(justify right)
-				(hide yes)
-			)
-		)
-	)
 	(global_label "AIRIN2"
 		(shape input)
@@
 		)
 	)
-	(global_label "ADC1"
-		(shape input)
-		(at 55.88 105.41 180)
-		(fields_autoplaced yes)
-		(effects
-			(font
-				(size 0.762 0.762)
-			)
-			(justify right)
-		)
-		(property "Intersheetrefs" "${INTERSHEET_REFS}"
-			(at 51.1858 105.41 0)
-			(effects
-				(font
-					(size 1.27 1.27)
-				)
-				(justify right)
-				(hide yes)
-			)
-		)
-	)
 	(global_label "SW1"
 		(shape input)
@@
 		)
 	)
+	(global_label "PWM3"
+		(shape input)
+		(at 166.37 55.88 180)
+		(fields_autoplaced yes)
+		(effects
+			(font
+				(size 0.762 0.762)
+			)
+			(justify right)
+		)
+		(property "Intersheetrefs" "${INTERSHEET_REFS}"
+			(at 161.3491 55.88 0)
+			(effects
+				(font
+					(size 1.27 1.27)
+				)
+				(justify right)
+				(hide yes)
+			)
+		)
+	)
 	(global_label "MOS_IN3"
 		(shape input)
@@
 				(hide yes)
 			)
+		)
+	)
+	(global_label "PWM4"
+		(shape input)
+		(at 166.37 58.42 180)
+		(fields_autoplaced yes)
+		(effects
+			(font
+				(size 0.762 0.762)
+			)
+			(justify right)
+		)
+		(property "Intersheetrefs" "${INTERSHEET_REFS}"
+			(at 161.3491 58.42 0)
+			(effects
+				(font
+					(size 1.27 1.27)
+				)
+				(justify right)
+				(hide yes)
+			)
